File: KiCad_PCB/SdraKb00.kicad_sch (KiCad schematic)
At the start: 77 parts, among them J1 AVR-ISP-6, SW00 SW_Push_45deg, SW01 SW_Push_45deg, SW02 SW_Push_45deg, SW03 RotaryEncoder_Switch, SW10 SW_Push_45deg, SW11 SW_Push_45deg, SW12 SW_Push_45deg, SW13 SW_Push_45deg, SW20 SW_Push_45deg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

Commit message: Changing power indicator specs. (#10)
Parts:
- D4: value RED 1.8V -> RED 2V
- R10: value 640 -> 150
Changed lines of the file:
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@@
 			)
 		)
-		(property "Value" "640"
+		(property "Value" "150"
 			(at 247.65 147.3199 0)
 			(effects
@@
 			)
 		)
-		(property "Value" "RED 1.8V"
+		(property "Value" "RED 2V"
 			(at 250.698 152.4 0)
 			(effects
